File: microquad-v1/liion_bat.sch (KiCad schematic (older format))
At the start: 12 parts

Commit message: Changed IMU to I2C pins
Changed lines of the file:
@@
 $EndComp
 Wire Wire Line
-	5600 1800 5600 2250
+	5600 2100 5600 2250
 Wire Wire Line
 	5600 2250 5600 2750
@@
 Connection ~ 3500 4350
 Wire Wire Line
-	4325 1800 4325 2675
+	4325 2100 4325 2675
 Wire Wire Line
 	4325 2675 3500 2675
@@
 Connection ~ 5400 2750
 Wire Wire Line
-	4325 1800 5600 1800
+	4325 2100 5600 2100
 Wire Wire Line
 	5350 2850 5950 2850
