File: microquad-v1/liion_bat.sch (KiCad schematic (older format))
At the start: 10 parts

Commit message: Fixed DRC errors (the ladybug is now happy)
Parts:
- gave numbers to parts that had none: 10
Changed lines of the file:
@@
 $Descr A4 11693 8268
 encoding utf-8
-Sheet 5 8
+Sheet 5 9
 Title ""
 Date ""
@@
 P 4900 2900
 AR Path="/59F6680F/59F538F1" Ref="Ubat?"  Part="1"
-AR Path="/59F56F7F/59F538F1" Ref="Ubat?"  Part="1"
-F 0 "Ubat?" H 4650 3200 60  0000 L CNN
+AR Path="/59F56F7F/59F538F1" Ref="Ubat1"  Part="1"
+F 0 "Ubat1" H 4650 3200 60  0000 L CNN
 F 1 "TPS2112A" H 4650 2600 60  0000 L CNN
 F 2 "Housings_SSOP:TSSOP-8_4.4x3mm_Pitch0.65mm" H 4850 2900 60  0001 C CNN
@@
 P 5700 2400
 AR Path="/59F6680F/59F53938" Ref="Cbat?"  Part="1"
-AR Path="/59F56F7F/59F53938" Ref="Cbat?"  Part="1"
-F 0 "Cbat?" H 5710 2470 50  0000 L CNN
+AR Path="/59F56F7F/59F53938" Ref="Cbat3"  Part="1"
+F 0 "Cbat3" H 5710 2470 50  0000 L CNN
 F 1 "0.1uF" H 5710 2320 50  0000 L CNN
 F 2 "Capacitors_SMD:C_0603" H 5700 2400 50  0001 C CNN
@@
 P 5700 2550
 AR Path="/59F6680F/59F53940" Ref="#PWR019"  Part="1"
-AR Path="/59F56F7F/59F53940" Ref="#PWR019"  Part="1"
-F 0 "#PWR019" H 5700 2300 50  0001 C CNN
+AR Path="/59F56F7F/59F53940" Ref="#PWR030"  Part="1"
+F 0 "#PWR030" H 5700 2300 50  0001 C CNN
 F 1 "GND" H 5700 2400 50  0000 C CNN
 F 2 "" H 5700 2550 50  0001 C CNN
@@
 P 5425 3125
 AR Path="/59F6680F/59F5394A" Ref="#PWR020"  Part="1"
-AR Path="/59F56F7F/59F5394A" Ref="#PWR020"  Part="1"
-F 0 "#PWR020" H 5425 2875 50  0001 C CNN
+AR Path="/59F56F7F/59F5394A" Ref="#PWR031"  Part="1"
+F 0 "#PWR031" H 5425 2875 50  0001 C CNN
 F 1 "GND" H 5425 2975 50  0000 C CNN
 F 2 "" H 5425 3125 50  0001 C CNN
@@
 P 4400 3500
 AR Path="/59F6680F/59F53953" Ref="#PWR021"  Part="1"
-AR Path="/59F56F7F/59F53953" Ref="#PWR021"  Part="1"
-F 0 "#PWR021" H 4400 3250 50  0001 C CNN
+AR Path="/59F56F7F/59F53953" Ref="#PWR032"  Part="1"
+F 0 "#PWR032" H 4400 3250 50  0001 C CNN
 F 1 "GND" H 4400 3350 50  0000 C CNN
 F 2 "" H 4400 3500 50  0001 C CNN
@@
 P 4400 3300
 AR Path="/59F6680F/59F5395B" Ref="Rbat?"  Part="1"
-AR Path="/59F56F7F/59F5395B" Ref="Rbat?"  Part="1"
-F 0 "Rbat?" V 4480 3300 50  0000 C CNN
+AR Path="/59F56F7F/59F5395B" Ref="Rbat2"  Part="1"
+F 0 "Rbat2" V 4480 3300 50  0000 C CNN
 F 1 "402" V 4400 3300 50  0000 C CNN
 F 2 "Resistors_SMD:R_0603" V 4330 3300 50  0001 C CNN
@@
 P 4825 3800
 AR Path="/59F6680F/59F5396D" Ref="Jbat?"  Part="1"
-AR Path="/59F56F7F/59F5396D" Ref="Jbat?"  Part="1"
-F 0 "Jbat?" H 4825 3900 50  0000 C CNN
+AR Path="/59F56F7F/59F5396D" Ref="Jbat1"  Part="1"
+F 0 "Jbat1" H 4825 3900 50  0000 C CNN
 F 1 "Battery 1x2" H 4825 3600 50  0000 C CNN
 F 2 "Connectors_JST:JST_PH_S2B-PH-SM4-TB_02x2.00mm_Angled" H 4825 3800 50  0001 C CNN
@@
 P 5100 3950
 AR Path="/59F6680F/59F53974" Ref="#PWR022"  Part="1"
-AR Path="/59F56F7F/59F53974" Ref="#PWR022"  Part="1"
-F 0 "#PWR022" H 5100 3700 50  0001 C CNN
+AR Path="/59F56F7F/59F53974" Ref="#PWR033"  Part="1"
+F 0 "#PWR033" H 5100 3700 50  0001 C CNN
 F 1 "GND" H 5100 3800 50  0000 C CNN
 F 2 "" H 5100 3950 50  0001 C CNN
@@
 P 5425 4800
 AR Path="/59F6680F/59F53983" Ref="Cbat?"  Part="1"
-AR Path="/59F56F7F/59F53983" Ref="Cbat?"  Part="1"
-F 0 "Cbat?" H 5435 4870 50  0000 L CNN
+AR Path="/59F56F7F/59F53983" Ref="Cbat2"  Part="1"
+F 0 "Cbat2" H 5435 4870 50  0000 L CNN
 F 1 "1uF" H 5435 4720 50  0000 L CNN
 F 2 "Capacitors_SMD:C_0603" H 5425 4800 50  0001 C CNN
@@
 P 5425 4975
 AR Path="/59F6680F/59F5398C" Ref="#PWR023"  Part="1"
-AR Path="/59F56F7F/59F5398C" Ref="#PWR023"  Part="1"
-F 0 "#PWR023" H 5425 4725 50  0001 C CNN
+AR Path="/59F56F7F/59F5398C" Ref="#PWR034"  Part="1"
+F 0 "#PWR034" H 5425 4725 50  0001 C CNN
 F 1 "GND" H 5425 4825 50  0000 C CNN
 F 2 "" H 5425 4975 50  0001 C CNN
@@
 P 4975 5075
 AR Path="/59F6680F/59F53993" Ref="#PWR024"  Part="1"
-AR Path="/59F56F7F/59F53993" Ref="#PWR024"  Part="1"
-F 0 "#PWR024" H 4975 4825 50  0001 C CNN
+AR Path="/59F56F7F/59F53993" Ref="#PWR035"  Part="1"
+F 0 "#PWR035" H 4975 4825 50  0001 C CNN
 F 1 "GND" H 4975 4925 50  0000 C CNN
 F 2 "" H 4975 5075 50  0001 C CNN
@@
 P 5075 4875
 AR Path="/59F6680F/59F5399C" Ref="Rbat?"  Part="1"
-AR Path="/59F56F7F/59F5399C" Ref="Rbat?"  Part="1"
-F 0 "Rbat?" H 5105 4895 50  0000 L CNN
+AR Path="/59F56F7F/59F5399C" Ref="Rbat3"  Part="1"
+F 0 "Rbat3" H 5105 4895 50  0000 L CNN
 F 1 "2K" H 5105 4835 50  0000 L CNN
 F 2 "Resistors_SMD:R_0603" H 5075 4875 50  0001 C CNN
@@
 	3925 4350 3925 4850
 Wire Wire Line
-	3925 4350 3500 4350
+	3500 4350 3925 4350
 $Comp
 L C_Small Cbat?
@@
 P 3700 4500
 AR Path="/59F6680F/59F539BD" Ref="Cbat?"  Part="1"
-AR Path="/59F56F7F/59F539BD" Ref="Cbat?"  Part="1"
-F 0 "Cbat?" H 3710 4570 50  0000 L CNN
+AR Path="/59F56F7F/59F539BD" Ref="Cbat1"  Part="1"
+F 0 "Cbat1" H 3710 4570 50  0000 L CNN
 F 1 "1uF" H 3710 4420 50  0000 L CNN
 F 2 "Capacitors_SMD:C_0603" H 3700 4500 50  0001 C CNN
@@
 P 3700 4650
 AR Path="/59F6680F/59F539C4" Ref="#PWR025"  Part="1"
-AR Path="/59F56F7F/59F539C4" Ref="#PWR025"  Part="1"
-F 0 "#PWR025" H 3700 4400 50  0001 C CNN
+AR Path="/59F56F7F/59F539C4" Ref="#PWR036"  Part="1"
+F 0 "#PWR036" H 3700 4400 50  0001 C CNN
 F 1 "GND" H 3800 4550 50  0000 C CNN
 F 2 "" H 3700 4650 50  0001 C CNN
@@
 P 4875 2450
 AR Path="/59F6680F/59F53A15" Ref="R?"  Part="1"
-AR Path="/59F56F7F/59F53A15" Ref="R?"  Part="1"
-F 0 "R?" V 4955 2450 50  0000 C CNN
+AR Path="/59F56F7F/59F53A15" Ref="R6"  Part="1"
+F 0 "R6" V 4955 2450 50  0000 C CNN
 F 1 "20K" V 4875 2450 50  0000 C CNN
 F 2 "Resistors_SMD:R_0603" V 4805 2450 50  0001 C CNN
@@
 P 4250 3300
 AR Path="/59F6680F/59F53A1D" Ref="Rbat?"  Part="1"
-AR Path="/59F56F7F/59F53A1D" Ref="Rbat?"  Part="1"
-F 0 "Rbat?" V 4330 3300 50  0000 C CNN
+AR Path="/59F56F7F/59F53A1D" Ref="Rbat1"  Part="1"
+F 0 "Rbat1" V 4330 3300 50  0000 C CNN
 F 1 "10K" V 4250 3300 50  0000 C CNN
 F 2 "Resistors_SMD:R_0603" V 4180 3300 50  0001 C CNN
@@
 P 4025 2925
 AR Path="/59F6680F/59F53A24" Ref="#PWR026"  Part="1"
-AR Path="/59F56F7F/59F53A24" Ref="#PWR026"  Part="1"
-F 0 "#PWR026" H 4025 2675 50  0001 C CNN
+AR Path="/59F56F7F/59F53A24" Ref="#PWR037"  Part="1"
+F 0 "#PWR037" H 4025 2675 50  0001 C CNN
 F 1 "GND" H 4025 2775 50  0000 C CNN
 F 2 "" H 4025 2925 50  0001 C CNN
@@
 P 4250 3500
 AR Path="/59F6680F/59F53A2D" Ref="#PWR027"  Part="1"
-AR Path="/59F56F7F/59F53A2D" Ref="#PWR027"  Part="1"
-F 0 "#PWR027" H 4250 3250 50  0001 C CNN
+AR Path="/59F56F7F/59F53A2D" Ref="#PWR038"  Part="1"
+F 0 "#PWR038" H 4250 3250 50  0001 C CNN
 F 1 "GND" H 4250 3350 50  0000 C CNN
 F 2 "" H 4250 3500 50  0001 C CNN
@@
 	4325 1800 5600 1800
 Wire Wire Line
-	5350 2850 5950 2850
-Text HLabel 5950 2850 2    60   Input ~ 0
+	5350 2850 6275 2850
+Text HLabel 6275 2850 2    60   Input ~ 0
 Vout
 Text HLabel 3500 2675 0    60   Input ~ 0
@@
 Origionally layed out by Alex Hoppe and others.\nhttps://github.com/aehoppe/E70N19_Dev_Board\nEdited by Marie-Caroline to switch Battery Charger
 $Comp
-L MCP73812T U?
+L MCP73812T U4
 U 1 1 59F66E7B
 P 4450 4750
-F 0 "U?" H 4200 5000 60  0000 L CNN
+F 0 "U4" H 4200 5000 60  0000 L CNN
 F 1 "MCP73812T" H 4200 4500 60  0000 L CNN
 F 2 "" H 4450 4750 60  0001 C CNN

Commit message: Notes from schematic review
Changed lines of the file:
@@
 $EndComp
 Wire Wire Line
-	5600 2750 5350 2750
+	5600 2750 5400 2750
+Wire Wire Line
+	5400 2750 5350 2750
 $Comp
 L C_Small Cbat?
@@
 $EndComp
 Wire Wire Line
-	5600 1800 5600 2750
+	5600 2150 5600 2250
+Wire Wire Line
+	5600 2250 5600 2750
 $Comp
 L GND #PWR019
@@
 P 5700 2550
 AR Path="/59F6680F/59F53940" Ref="#PWR019"  Part="1"
-AR Path="/59F56F7F/59F53940" Ref="#PWR030"  Part="1"
-F 0 "#PWR030" H 5700 2300 50  0001 C CNN
+AR Path="/59F56F7F/59F53940" Ref="#PWR029"  Part="1"
+F 0 "#PWR029" H 5700 2300 50  0001 C CNN
 F 1 "GND" H 5700 2400 50  0000 C CNN
 F 2 "" H 5700 2550 50  0001 C CNN
@@
 P 5425 3125
 AR Path="/59F6680F/59F5394A" Ref="#PWR020"  Part="1"
-AR Path="/59F56F7F/59F5394A" Ref="#PWR031"  Part="1"
-F 0 "#PWR031" H 5425 2875 50  0001 C CNN
+AR Path="/59F56F7F/59F5394A" Ref="#PWR030"  Part="1"
+F 0 "#PWR030" H 5425 2875 50  0001 C CNN
 F 1 "GND" H 5425 2975 50  0000 C CNN
 F 2 "" H 5425 3125 50  0001 C CNN
@@
 P 4400 3500
 AR Path="/59F6680F/59F53953" Ref="#PWR021"  Part="1"
-AR Path="/59F56F7F/59F53953" Ref="#PWR032"  Part="1"
-F 0 "#PWR032" H 4400 3250 50  0001 C CNN
+AR Path="/59F56F7F/59F53953" Ref="#PWR031"  Part="1"
+F 0 "#PWR031" H 4400 3250 50  0001 C CNN
 F 1 "GND" H 4400 3350 50  0000 C CNN
 F 2 "" H 4400 3500 50  0001 C CNN
@@
 P 5100 3950
 AR Path="/59F6680F/59F53974" Ref="#PWR022"  Part="1"
-AR Path="/59F56F7F/59F53974" Ref="#PWR033"  Part="1"
-F 0 "#PWR033" H 5100 3700 50  0001 C CNN
+AR Path="/59F56F7F/59F53974" Ref="#PWR032"  Part="1"
+F 0 "#PWR032" H 5100 3700 50  0001 C CNN
 F 1 "GND" H 5100 3800 50  0000 C CNN
 F 2 "" H 5100 3950 50  0001 C CNN
@@
 $EndComp
 Wire Wire Line
-	5025 3800 5625 3800
+	5025 3800 5450 3800
+Wire Wire Line
+	5450 3800 5625 3800
 Wire Wire Line
 	5625 3800 5625 2950
@@
 	5100 3900 5100 3950
 Wire Wire Line
-	4900 4650 5450 4650
+	4900 4650 5425 4650
+Wire Wire Line
+	5425 4650 5450 4650
 Wire Wire Line
 	5450 4650 5450 3800
@@
 P 5425 4975
 AR Path="/59F6680F/59F5398C" Ref="#PWR023"  Part="1"
-AR Path="/59F56F7F/59F5398C" Ref="#PWR034"  Part="1"
-F 0 "#PWR034" H 5425 4725 50  0001 C CNN
+AR Path="/59F56F7F/59F5398C" Ref="#PWR033"  Part="1"
+F 0 "#PWR033" H 5425 4725 50  0001 C CNN
 F 1 "GND" H 5425 4825 50  0000 C CNN
 F 2 "" H 5425 4975 50  0001 C CNN
@@
 P 4975 5075
 AR Path="/59F6680F/59F53993" Ref="#PWR024"  Part="1"
-AR Path="/59F56F7F/59F53993" Ref="#PWR035"  Part="1"
-F 0 "#PWR035" H 4975 4825 50  0001 C CNN
+AR Path="/59F56F7F/59F53993" Ref="#PWR034"  Part="1"
+F 0 "#PWR034" H 4975 4825 50  0001 C CNN
 F 1 "GND" H 4975 4925 50  0000 C CNN
 F 2 "" H 4975 5075 50  0001 C CNN
@@
 	4900 4850 4975 4850
 Wire Wire Line
-	4975 4850 4975 5075
+	4975 4850 4975 5025
+Wire Wire Line
+	4975 5025 4975 5075
 $Comp
 L R_Small Rbat?
@@
 	4000 4650 3925 4650
 Wire Wire Line
-	3925 4350 3925 4850
-Wire Wire Line
-	3500 4350 3925 4350
+	3925 4350 3925 4650
+Wire Wire Line
+	3925 4650 3925 4850
+Wire Wire Line
+	3500 4350 3700 4350
+Wire Wire Line
+	3700 4350 3925 4350
 $Comp
 L C_Small Cbat?
@@
 P 3700 4650
 AR Path="/59F6680F/59F539C4" Ref="#PWR025"  Part="1"
-AR Path="/59F56F7F/59F539C4" Ref="#PWR036"  Part="1"
-F 0 "#PWR036" H 3700 4400 50  0001 C CNN
+AR Path="/59F56F7F/59F539C4" Ref="#PWR035"  Part="1"
+F 0 "#PWR035" H 3700 4400 50  0001 C CNN
 F 1 "GND" H 3800 4550 50  0000 C CNN
 F 2 "" H 3700 4650 50  0001 C CNN
@@
 Connection ~ 3700 4350
 Wire Wire Line
-	4325 1800 4325 2675
+	4325 2150 4325 2675
 Wire Wire Line
 	4325 2675 3500 2675
@@
 P 4025 2925
 AR Path="/59F6680F/59F53A24" Ref="#PWR026"  Part="1"
-AR Path="/59F56F7F/59F53A24" Ref="#PWR037"  Part="1"
-F 0 "#PWR037" H 4025 2675 50  0001 C CNN
+AR Path="/59F56F7F/59F53A24" Ref="#PWR036"  Part="1"
+F 0 "#PWR036" H 4025 2675 50  0001 C CNN
 F 1 "GND" H 4025 2775 50  0000 C CNN
 F 2 "" H 4025 2925 50  0001 C CNN
@@
 	4250 3150 4250 2950
 Wire Wire Line
-	4250 2950 4450 2950
+	4250 2950 4375 2950
+Wire Wire Line
+	4375 2950 4450 2950
 $Comp
 L GND #PWR027
@@
 P 4250 3500
 AR Path="/59F6680F/59F53A2D" Ref="#PWR027"  Part="1"
-AR Path="/59F56F7F/59F53A2D" Ref="#PWR038"  Part="1"
-F 0 "#PWR038" H 4250 3250 50  0001 C CNN
+AR Path="/59F56F7F/59F53A2D" Ref="#PWR037"  Part="1"
+F 0 "#PWR037" H 4250 3250 50  0001 C CNN
 F 1 "GND" H 4250 3350 50  0000 C CNN
 F 2 "" H 4250 3500 50  0001 C CNN
@@
 Connection ~ 5400 2750
 Wire Wire Line
-	4325 1800 5600 1800
+	4325 2150 5600 2150
 Wire Wire Line
 	5350 2850 6275 2850
@@
 U 1 1 59F66E7B
 P 4450 4750
+AR Path="/59F66E7B" Ref="U4"  Part="1"
+AR Path="/59F56F7F/59F66E7B" Ref="U4"  Part="1"
 F 0 "U4" H 4200 5000 60  0000 L CNN
 F 1 "MCP73812T" H 4200 4500 60  0000 L CNN

Commit message: Added layout for transistor
Changed lines of the file:
@@
 $EndComp
 Wire Wire Line
-	5600 2750 5400 2750
-Wire Wire Line
-	5400 2750 5350 2750
+	5600 2750 5350 2750
 $Comp
 L C_Small Cbat?
@@
 $EndComp
 Wire Wire Line
-	5600 2150 5600 2250
-Wire Wire Line
-	5600 2250 5600 2750
+	5600 2150 5600 2750
 $Comp
 L GND #PWR019
@@
 P 5700 2550
 AR Path="/59F6680F/59F53940" Ref="#PWR019"  Part="1"
-AR Path="/59F56F7F/59F53940" Ref="#PWR30"  Part="1"
-F 0 "#PWR30" H 5700 2300 50  0001 C CNN
+AR Path="/59F56F7F/59F53940" Ref="#PWR024"  Part="1"
+F 0 "#PWR024" H 5700 2300 50  0001 C CNN
 F 1 "GND" H 5700 2400 50  0000 C CNN
 F 2 "" H 5700 2550 50  0001 C CNN
@@
 P 5425 3125
 AR Path="/59F6680F/59F5394A" Ref="#PWR020"  Part="1"
-AR Path="/59F56F7F/59F5394A" Ref="#PWR28"  Part="1"
-F 0 "#PWR28" H 5425 2875 50  0001 C CNN
+AR Path="/59F56F7F/59F5394A" Ref="#PWR025"  Part="1"
+F 0 "#PWR025" H 5425 2875 50  0001 C CNN
 F 1 "GND" H 5425 2975 50  0000 C CNN
 F 2 "" H 5425 3125 50  0001 C CNN
@@
 P 4400 3500
 AR Path="/59F6680F/59F53953" Ref="#PWR021"  Part="1"
-AR Path="/59F56F7F/59F53953" Ref="#PWR25"  Part="1"
-F 0 "#PWR25" H 4400 3250 50  0001 C CNN
+AR Path="/59F56F7F/59F53953" Ref="#PWR026"  Part="1"
+F 0 "#PWR026" H 4400 3250 50  0001 C CNN
 F 1 "GND" H 4400 3350 50  0000 C CNN
 F 2 "" H 4400 3500 50  0001 C CNN
@@
 P 5100 3950
 AR Path="/59F6680F/59F53974" Ref="#PWR022"  Part="1"
-AR Path="/59F56F7F/59F53974" Ref="#PWR27"  Part="1"
-F 0 "#PWR27" H 5100 3700 50  0001 C CNN
+AR Path="/59F56F7F/59F53974" Ref="#PWR027"  Part="1"
+F 0 "#PWR027" H 5100 3700 50  0001 C CNN
 F 1 "GND" H 5100 3800 50  0000 C CNN
 F 2 "" H 5100 3950 50  0001 C CNN
@@
 $EndComp
 Wire Wire Line
-	5025 3800 5450 3800
-Wire Wire Line
-	5450 3800 5625 3800
+	5025 3800 5625 3800
 Wire Wire Line
 	5625 3800 5625 2950
@@
 	5100 3900 5100 3950
 Wire Wire Line
-	4900 4650 5425 4650
-Wire Wire Line
-	5425 4650 5450 4650
+	4900 4650 5450 4650
 Wire Wire Line
 	5450 4650 5450 3800
@@
 P 5425 4975
 AR Path="/59F6680F/59F5398C" Ref="#PWR023"  Part="1"
-AR Path="/59F56F7F/59F5398C" Ref="#PWR29"  Part="1"
-F 0 "#PWR29" H 5425 4725 50  0001 C CNN
+AR Path="/59F56F7F/59F5398C" Ref="#PWR028"  Part="1"
+F 0 "#PWR028" H 5425 4725 50  0001 C CNN
 F 1 "GND" H 5425 4825 50  0000 C CNN
 F 2 "" H 5425 4975 50  0001 C CNN
@@
 P 4975 5075
 AR Path="/59F6680F/59F53993" Ref="#PWR024"  Part="1"
-AR Path="/59F56F7F/59F53993" Ref="#PWR26"  Part="1"
-F 0 "#PWR26" H 4975 4825 50  0001 C CNN
+AR Path="/59F56F7F/59F53993" Ref="#PWR029"  Part="1"
+F 0 "#PWR029" H 4975 4825 50  0001 C CNN
 F 1 "GND" H 4975 4925 50  0000 C CNN
 F 2 "" H 4975 5075 50  0001 C CNN
@@
 	4900 4850 4975 4850
 Wire Wire Line
-	4975 4850 4975 5025
-Wire Wire Line
-	4975 5025 4975 5075
+	4975 4850 4975 5075
 $Comp
 L R_Small Rbat?
@@
 	4000 4650 3925 4650
 Wire Wire Line
-	3925 4350 3925 4650
-Wire Wire Line
-	3925 4650 3925 4850
-Wire Wire Line
-	3500 4350 3700 4350
-Wire Wire Line
-	3700 4350 3925 4350
+	3925 4350 3925 4850
+Wire Wire Line
+	3500 4350 3925 4350
 $Comp
 L C_Small Cbat?
@@
 P 3700 4650
 AR Path="/59F6680F/59F539C4" Ref="#PWR025"  Part="1"
-AR Path="/59F56F7F/59F539C4" Ref="#PWR22"  Part="1"
-F 0 "#PWR22" H 3700 4400 50  0001 C CNN
+AR Path="/59F56F7F/59F539C4" Ref="#PWR030"  Part="1"
+F 0 "#PWR030" H 3700 4400 50  0001 C CNN
 F 1 "GND" H 3800 4550 50  0000 C CNN
 F 2 "" H 3700 4650 50  0001 C CNN
@@
 P 4025 2925
 AR Path="/59F6680F/59F53A24" Ref="#PWR026"  Part="1"
-AR Path="/59F56F7F/59F53A24" Ref="#PWR23"  Part="1"
-F 0 "#PWR23" H 4025 2675 50  0001 C CNN
+AR Path="/59F56F7F/59F53A24" Ref="#PWR031"  Part="1"
+F 0 "#PWR031" H 4025 2675 50  0001 C CNN
 F 1 "GND" H 4025 2775 50  0000 C CNN
 F 2 "" H 4025 2925 50  0001 C CNN
@@
 	4250 3150 4250 2950
 Wire Wire Line
-	4250 2950 4375 2950
-Wire Wire Line
-	4375 2950 4450 2950
+	4250 2950 4450 2950
 $Comp
 L GND #PWR027
@@
 P 4250 3500
 AR Path="/59F6680F/59F53A2D" Ref="#PWR027"  Part="1"
-AR Path="/59F56F7F/59F53A2D" Ref="#PWR24"  Part="1"
-F 0 "#PWR24" H 4250 3250 50  0001 C CNN
+AR Path="/59F56F7F/59F53A2D" Ref="#PWR032"  Part="1"
+F 0 "#PWR032" H 4250 3250 50  0001 C CNN
 F 1 "GND" H 4250 3350 50  0000 C CNN
 F 2 "" H 4250 3500 50  0001 C CNN

Commit message: Finished footprint work 10/31
Parts:
- U4: footprint (none) -> TO_SOT_Packages_SMD:SOT-23
Changed lines of the file:
@@
 F 0 "U4" H 4200 5000 60  0000 L CNN
 F 1 "MCP73812T" H 4200 4500 60  0000 L CNN
-F 2 "" H 4450 4750 60  0001 C CNN
+F 2 "TO_SOT_Packages_SMD:SOT-23" H 4450 4750 60  0001 C CNN
 F 3 "" H 4450 4750 60  0001 C CNN
 	1    4450 4750
