File: microquad-v1/mpu9250.sch (KiCad schematic (older format))
At the start: 4 parts

Commit message: Changed IMU to I2C pins
Connections:
- net CS is gone; now on net +3V3: Uimu?.22 (~CS)
- net SDO is gone; now on net GND: Uimu?.9 (AD0)
- net SCK renamed SCL
- net SDI renamed SDA
Changed lines of the file:
@@
 Wire Wire Line
 	6400 2600 6400 2800
-Text HLabel 4550 2600 0    60   Input ~ 0
-CS
 Text HLabel 4550 2800 0    60   Input ~ 0
-SCK
+SCL
 Text HLabel 4550 3000 0    60   Input ~ 0
-SDI
-Text HLabel 4550 3200 0    60   Input ~ 0
-SDO
+SDA
 Text HLabel 4550 3400 0    60   Input ~ 0
 INT
@@
 Text Notes 4500 850  0    60   ~ 0
 Origionally from Brad's IMUlogger2
+Wire Wire Line
+	4550 2600 4550 2275
+Wire Wire Line
+	4550 2275 6350 2275
+Wire Wire Line
+	6350 2275 6350 2600
+$Comp
+L GND #PWR?
+U 1 1 59F6670B
+P 4550 3200
+F 0 "#PWR?" H 4550 2950 50  0001 C CNN
+F 1 "GND" H 4550 3050 50  0000 C CNN
+F 2 "" H 4550 3200 50  0001 C CNN
+F 3 "" H 4550 3200 50  0001 C CNN
+	1    4550 3200
+	0    1    1    0
+$EndComp
 $EndSCHEMATC
