File: microquad-v1/mpu9250.sch (KiCad schematic (older format))
At the start: 4 parts

Commit message: Fixed DRC errors (the ladybug is now happy)
Parts:
- gave numbers to parts that had none: 4
Changed lines of the file:
@@
 $Descr A4 11693 8268
 encoding utf-8
-Sheet 6 8
+Sheet 6 9
 Title ""
 Date ""
@@
 $EndDescr
 $Comp
-L MPU-9250A Uimu?
+L MPU-9250A Uimu1
 U 1 1 59F58674
 P 5450 3400
-F 0 "Uimu?" H 4750 4450 60  0000 L CNN
+F 0 "Uimu1" H 4750 4450 60  0000 L CNN
 F 1 "MPU-9250A" H 4750 4350 60  0000 L CNN
 F 2 "imulogger2:QFN40P300X300X105-25N" H 5450 4200 60  0001 C CNN
@@
 $EndComp
 $Comp
-L GND #PWR028
+L GND #PWR041
 U 1 1 59F5867B
 P 6400 4050
-F 0 "#PWR028" H 6400 3800 50  0001 C CNN
+F 0 "#PWR041" H 6400 3800 50  0001 C CNN
 F 1 "GND" H 6400 3900 50  0000 C CNN
 F 2 "" H 6400 4050 50  0001 C CNN
@@
 $EndComp
 $Comp
-L C Cimu?
+L C Cimu1
 U 1 1 59F58681
 P 6400 3400
-F 0 "Cimu?" H 6500 3400 50  0000 L CNN
+F 0 "Cimu1" H 6500 3400 50  0000 L CNN
 F 1 "0.1µF" H 6425 3300 50  0000 L CNN
 F 2 "Capacitors_SMD:C_0603" H 6438 3250 50  0001 C CNN
@@
 $EndComp
 $Comp
-L C Cimu?
+L C Cimu3
 U 1 1 59F58688
 P 6600 3000
-F 0 "Cimu?" V 6750 2950 50  0000 L CNN
+F 0 "Cimu3" V 6750 2950 50  0000 L CNN
 F 1 "0.1µF" H 6625 2900 50  0000 L CNN
 F 2 "Capacitors_SMD:C_0603" H 6638 2850 50  0001 C CNN
@@
 $EndComp
 $Comp
-L GND #PWR029
+L GND #PWR042
 U 1 1 59F5868F
 P 6850 3100
-F 0 "#PWR029" H 6850 2850 50  0001 C CNN
+F 0 "#PWR042" H 6850 2850 50  0001 C CNN
 F 1 "GND" H 6850 2950 50  0000 C CNN
 F 2 "" H 6850 3100 50  0001 C CNN
@@
 $EndComp
 $Comp
-L C Cimu?
+L C Cimu2
 U 1 1 59F58695
 P 6600 2600
-F 0 "Cimu?" V 6750 2550 50  0000 L CNN
+F 0 "Cimu2" V 6750 2550 50  0000 L CNN
 F 1 "10nF" H 6625 2500 50  0000 L CNN
 F 2 "Capacitors_SMD:C_0603" H 6638 2450 50  0001 C CNN
@@
 INT
 $Comp
-L +3V3 #PWR030
+L +3V3 #PWR043
 U 1 1 59F587B6
 P 6400 2600
-F 0 "#PWR030" H 6400 2450 50  0001 C CNN
+F 0 "#PWR043" H 6400 2450 50  0001 C CNN
 F 1 "+3V3" H 6400 2740 50  0000 C CNN
 F 2 "" H 6400 2600 50  0001 C CNN
@@
 $EndComp
 $Comp
-L +3V3 #PWR031
+L +3V3 #PWR044
 U 1 1 59F587D4
 P 6400 3000
-F 0 "#PWR031" H 6400 2850 50  0001 C CNN
+F 0 "#PWR044" H 6400 2850 50  0001 C CNN
 F 1 "+3V3" H 6400 3140 50  0000 C CNN
 F 2 "" H 6400 3000 50  0001 C CNN
@@
 	6350 2275 6350 2600
 $Comp
-L GND #PWR?
+L GND #PWR045
 U 1 1 59F6670B
 P 4550 3200
-F 0 "#PWR?" H 4550 2950 50  0001 C CNN
+F 0 "#PWR045" H 4550 2950 50  0001 C CNN
 F 1 "GND" H 4550 3050 50  0000 C CNN
 F 2 "" H 4550 3200 50  0001 C CNN
