File: microquad-v1/usb_uart.sch (KiCad schematic (older format))
At the start: 10 parts

Commit message: Changed IMU to I2C pins
Changed lines of the file:
@@
 $EndComp
 Wire Wire Line
-	4000 4475 4675 4475
-Wire Wire Line
-	4675 4475 4775 4475
-Wire Wire Line
-	4775 4475 4875 4475
+	4000 4475 4875 4475
 Connection ~ 4775 4475
 Wire Wire Line
@@
 	6400 4075 5475 4075
 Wire Wire Line
-	4000 3975 4000 4025
-Wire Wire Line
-	4000 4025 4000 4075
-Wire Wire Line
-	4000 4075 4000 4175
+	4000 3975 4000 4175
 Wire Wire Line
 	3775 3475 3775 3725
@@
 	3700 3525 3325 3525
 Wire Wire Line
-	2325 4425 2425 4425
-Wire Wire Line
-	2425 4425 2525 4425
-Wire Wire Line
-	2525 4425 2625 4425
-Wire Wire Line
-	2625 4425 2725 4425
-Wire Wire Line
-	2725 4425 2825 4425
-Wire Wire Line
-	2825 4425 2900 4425
+	2325 4425 2900 4425
 Wire Wire Line
 	2900 4425 2900 4475
@@
 Connection ~ 2825 4425
 Wire Wire Line
-	3325 3200 3450 3200
-Wire Wire Line
-	3450 3200 3575 3200
+	3325 3200 3575 3200
 Wire Wire Line
 	3325 3200 3325 3325
