File: microquad-v1/usb_uart.sch (KiCad schematic (older format))
At the start: 10 parts

Commit message: Changed LED resistor values
Parts:
- R? (x2): value 499 -> 1k
Changed lines of the file:
@@
 P 6400 3400
 F 0 "R?" V 6480 3400 50  0000 C CNN
-F 1 "499" V 6400 3400 50  0000 C CNN
+F 1 "1k" V 6400 3400 50  0000 C CNN
 F 2 "Resistors_SMD:R_0603" V 6330 3400 50  0001 C CNN
 F 3 "" H 6400 3400 50  0001 C CNN
@@
 P 6075 3400
 F 0 "R?" V 6155 3400 50  0000 C CNN
-F 1 "499" V 6075 3400 50  0000 C CNN
+F 1 "1k" V 6075 3400 50  0000 C CNN
 F 2 "Resistors_SMD:R_0603" V 6005 3400 50  0001 C CNN
 F 3 "" H 6075 3400 50  0001 C CNN
