File: microquad-v1/usb_uart.sch (KiCad schematic (older format))
At the start: 10 parts

Commit message: Fixed DRC errors (the ladybug is now happy)
Parts:
- gave numbers to parts that had none: 10
Changed lines of the file:
@@
 $Descr A4 11693 8268
 encoding utf-8
-Sheet 3 8
+Sheet 3 9
 Title ""
 Date ""
@@
 $EndDescr
 $Comp
-L FT230XS U?
+L FT230XS U3
 U 1 1 59F2772B
 P 4775 3775
-F 0 "U?" H 4225 4375 50  0000 L CNN
+F 0 "U3" H 4225 4375 50  0000 L CNN
 F 1 "FT230XS" H 5075 4375 50  0000 L CNN
 F 2 "Housings_SSOP:SSOP-16_3.9x4.9mm_Pitch0.635mm" H 4775 3775 50  0001 C CNN
@@
 $EndComp
 $Comp
-L GND #PWR05
+L GND #PWR016
 U 1 1 59F27732
 P 4775 4475
-F 0 "#PWR05" H 4775 4225 50  0001 C CNN
+F 0 "#PWR016" H 4775 4225 50  0001 C CNN
 F 1 "GND" H 4775 4325 50  0000 C CNN
 F 2 "" H 4775 4475 50  0001 C CNN
@@
 $EndComp
 $Comp
-L +3V3 #PWR06
+L +3V3 #PWR017
 U 1 1 59F27738
 P 3900 4025
-F 0 "#PWR06" H 3900 3875 50  0001 C CNN
+F 0 "#PWR017" H 3900 3875 50  0001 C CNN
 F 1 "+3V3" H 3900 4165 50  0000 C CNN
 F 2 "" H 3900 4025 50  0001 C CNN
@@
 $EndComp
 $Comp
-L R R?
+L R R2
 U 1 1 59F2773E
 P 3925 3475
-F 0 "R?" V 4005 3475 50  0000 C CNN
+F 0 "R2" V 4005 3475 50  0000 C CNN
 F 1 "30.1" V 3925 3475 50  0000 C CNN
 F 2 "Resistors_SMD:R_0603" V 3855 3475 50  0001 C CNN
@@
 $EndComp
 $Comp
-L R R?
+L R R1
 U 1 1 59F27745
 P 3925 3375
-F 0 "R?" V 4005 3375 50  0000 C CNN
+F 0 "R1" V 4005 3375 50  0000 C CNN
 F 1 "30.1" V 3925 3375 50  0000 C CNN
 F 2 "Resistors_SMD:R_0603" V 3855 3375 50  0001 C CNN
@@
 $EndComp
 $Comp
-L C C?
+L C C2
 U 1 1 59F2774C
 P 4000 4325
-F 0 "C?" H 4025 4425 50  0000 L CNN
+F 0 "C2" H 4025 4425 50  0000 L CNN
 F 1 "100nF" H 4025 4225 50  0000 L CNN
 F 2 "Capacitors_SMD:C_0603" H 4038 4175 50  0001 C CNN
@@
 $EndComp
 $Comp
-L LED Dtx?
+L LED Dtx1
 U 1 1 59F27753
 P 6075 3700
-F 0 "Dtx?" H 6075 3800 50  0000 C CNN
+F 0 "Dtx1" H 6075 3800 50  0000 C CNN
 F 1 "LED-G" H 6075 3600 50  0000 C CNN
 F 2 "LEDs:LED_0805" H 6075 3700 50  0001 C CNN
@@
 $EndComp
 $Comp
-L LED Drx?
+L LED Drx1
 U 1 1 59F2775A
 P 6400 3700
-F 0 "Drx?" H 6400 3800 50  0000 C CNN
+F 0 "Drx1" H 6400 3800 50  0000 C CNN
 F 1 "LED-G" H 6400 3600 50  0000 C CNN
 F 2 "LEDs:LED_0805" H 6400 3700 50  0001 C CNN
@@
 $EndComp
 $Comp
-L +3V3 #PWR07
+L +3V3 #PWR018
 U 1 1 59F27761
 P 6075 3250
-F 0 "#PWR07" H 6075 3100 50  0001 C CNN
+F 0 "#PWR018" H 6075 3100 50  0001 C CNN
 F 1 "+3V3" H 6075 3390 50  0000 C CNN
 F 2 "" H 6075 3250 50  0001 C CNN
@@
 $EndComp
 $Comp
-L +3V3 #PWR08
+L +3V3 #PWR019
 U 1 1 59F27767
 P 6400 3250
-F 0 "#PWR08" H 6400 3100 50  0001 C CNN
+F 0 "#PWR019" H 6400 3100 50  0001 C CNN
 F 1 "+3V3" H 6400 3390 50  0000 C CNN
 F 2 "" H 6400 3250 50  0001 C CNN
@@
 TX indicator
 $Comp
-L USB_microB_2040002-1 J?
+L USB_microB_2040002-1 J1
 U 1 1 59F27774
 P 2675 3725
-F 0 "J?" H 2225 4375 60  0000 L CNN
+F 0 "J1" H 2225 4375 60  0000 L CNN
 F 1 "USB_microB_2040002-1" H 2150 4275 60  0000 L CNN
 F 2 "USB_micro_b:USB_microB_2040002-1_alt" H 3025 3875 50  0001 C CNN
@@
 $EndComp
 $Comp
-L GND #PWR09
+L GND #PWR020
 U 1 1 59F2777B
 P 3325 4125
-F 0 "#PWR09" H 3325 3875 50  0001 C CNN
+F 0 "#PWR020" H 3325 3875 50  0001 C CNN
 F 1 "GND" H 3325 3975 50  0000 C CNN
 F 2 "" H 3325 4125 50  0001 C CNN
@@
 $EndComp
 $Comp
-L GS2 J?
+L GS2 J2
 U 1 1 59F27782
 P 3525 3925
-F 0 "J?" H 3450 3925 50  0000 C CNN
+F 0 "J2" H 3450 3925 50  0000 C CNN
 F 1 "GS2" H 3625 3776 50  0000 C CNN
 F 2 "Connectors:GS2" V 3599 3925 50  0001 C CNN
@@
 $EndComp
 $Comp
-L GND #PWR010
+L GND #PWR021
 U 1 1 59F27789
 P 3725 3925
-F 0 "#PWR010" H 3725 3675 50  0001 C CNN
+F 0 "#PWR021" H 3725 3675 50  0001 C CNN
 F 1 "GND" H 3725 3775 50  0000 C CNN
 F 2 "" H 3725 3925 50  0001 C CNN
@@
 $EndComp
 $Comp
-L R R?
+L R R4
 U 1 1 59F2778F
 P 6400 3400
-F 0 "R?" V 6480 3400 50  0000 C CNN
+F 0 "R4" V 6480 3400 50  0000 C CNN
 F 1 "1k" V 6400 3400 50  0000 C CNN
 F 2 "Resistors_SMD:R_0603" V 6330 3400 50  0001 C CNN
@@
 $EndComp
 $Comp
-L R R?
+L R R3
 U 1 1 59F27796
 P 6075 3400
-F 0 "R?" V 6155 3400 50  0000 C CNN
+F 0 "R3" V 6155 3400 50  0000 C CNN
 F 1 "1k" V 6075 3400 50  0000 C CNN
 F 2 "Resistors_SMD:R_0603" V 6005 3400 50  0001 C CNN
@@
 $EndComp
 $Comp
-L GND #PWR011
+L GND #PWR022
 U 1 1 59F2779D
 P 2900 4475
-F 0 "#PWR011" H 2900 4225 50  0001 C CNN
+F 0 "#PWR022" H 2900 4225 50  0001 C CNN
 F 1 "GND" H 2900 4325 50  0000 C CNN
 F 2 "" H 2900 4475 50  0001 C CNN
@@
 $EndComp
 $Comp
-L PWR_FLAG #FLG012
-U 1 1 59F277A3
-P 3450 3200
-F 0 "#FLG012" H 3450 3275 50  0001 C CNN
-F 1 "PWR_FLAG" H 3450 3350 50  0000 C CNN
-F 2 "" H 3450 3200 50  0001 C CNN
-F 3 "" H 3450 3200 50  0001 C CNN
-	1    3450 3200
-	1    0    0    -1
-$EndComp
-$Comp
-L PWR_FLAG #FLG013
+L PWR_FLAG #FLG024
 U 1 1 59F277A9
 P 3625 4500
-F 0 "#FLG013" H 3625 4575 50  0001 C CNN
+F 0 "#FLG024" H 3625 4575 50  0001 C CNN
 F 1 "PWR_FLAG" H 3625 4650 50  0000 C CNN
 F 2 "" H 3625 4500 50  0001 C CNN
@@
 $EndComp
 $Comp
-L GND #PWR014
+L GND #PWR025
 U 1 1 59F277AF
 P 3625 4500
-F 0 "#PWR014" H 3625 4250 50  0001 C CNN
+F 0 "#PWR025" H 3625 4250 50  0001 C CNN
 F 1 "GND" H 3625 4350 50  0000 C CNN
 F 2 "" H 3625 4500 50  0001 C CNN
@@
 Wire Wire Line
 	3325 3200 3325 3325
-Connection ~ 3450 3200
 NoConn ~ 5475 3575
 NoConn ~ 5475 3675

Commit message: Added footprint library for USB connector and BT chip
Parts:
- J1: footprint USB_micro_b:USB_microB_2040002-1_alt -> eclectronics:USB_microB_2040002-1
Changed lines of the file:
@@
 F 0 "J1" H 2225 4375 60  0000 L CNN
 F 1 "USB_microB_2040002-1" H 2150 4275 60  0000 L CNN
-F 2 "USB_micro_b:USB_microB_2040002-1_alt" H 3025 3875 50  0001 C CNN
+F 2 "eclectronics:USB_microB_2040002-1" H 3025 3875 50  0001 C CNN
 F 3 "" H 3025 3875 50  0001 C CNN
 	1    2675 3725

Commit message: Finished in-class work 10/2
Parts:
- removed J2: GS2, Connectors:GS2, symbol GS2
Changed lines of the file:
@@
-$EndComp
-$Comp
-L GS2 J2
-U 1 1 59F27782
-P 3525 3925
-F 0 "J2" H 3450 3925 50  0000 C CNN
-F 1 "GS2" H 3625 3776 50  0000 C CNN
-F 2 "Connectors:GS2" V 3599 3925 50  0001 C CNN
-F 3 "" H 3525 3925 50  0001 C CNN
-	1    3525 3925
-	0    1    1    0
-$EndComp
-$Comp
-L GND #PWR016
-U 1 1 59F27789
-P 3725 3925
-F 0 "#PWR016" H 3725 3675 50  0001 C CNN
-F 1 "GND" H 3725 3775 50  0000 C CNN
-F 2 "" H 3725 3925 50  0001 C CNN
-F 3 "" H 3725 3925 50  0001 C CNN
-	1    3725 3925
-	1    0    0    -1
 $EndComp
 $Comp
