File: microquad-v1/atmega328_power.sch (KiCad schematic (older format))
At the start: 6 parts

Commit message: Added reset button
Changed lines of the file:
@@
 $EndComp
 Wire Wire Line
-	1400 2650 1750 2650
-Wire Wire Line
-	1750 2650 2100 2650
-Wire Wire Line
-	2100 2650 2450 2650
+	1400 2650 2450 2650
 $Comp
 L C BC?
@@
 $EndComp
 Wire Wire Line
-	1500 3400 1650 3400
-Wire Wire Line
-	1650 3400 1800 3400
+	1500 3400 1800 3400
 $Comp
 L R R?
@@
 Connection ~ 1650 3400
 Wire Wire Line
-	1300 3700 1500 3700
-Wire Wire Line
-	1500 3700 1800 3700
+	1300 3700 1800 3700
 Connection ~ 1500 3700
 $EndSCHEMATC
