File: microquad-v1/atmega328_power.sch (KiCad schematic (older format))
At the start: 6 parts

Commit message: Fixed DRC errors (the ladybug is now happy)
Parts:
- gave numbers to parts that had none: 6
Changed lines of the file:
@@
 $Descr A4 11693 8268
 encoding utf-8
-Sheet 4 8
+Sheet 4 9
 Title ""
 Date ""
@@
 $EndDescr
 $Comp
-L C BC?
+L C BC1
 U 1 1 59F24977
 P 1400 2500
-F 0 "BC?" H 1425 2600 50  0000 L CNN
+F 0 "BC1" H 1425 2600 50  0000 L CNN
 F 1 "100nF" H 1425 2400 50  0000 L CNN
 F 2 "Capacitors_SMD:C_0603" H 1438 2350 50  0001 C CNN
@@
 $EndComp
 $Comp
-L GND #PWR015
+L GND #PWR026
 U 1 1 59F24A53
 P 1400 2800
-F 0 "#PWR015" H 1400 2550 50  0001 C CNN
+F 0 "#PWR026" H 1400 2550 50  0001 C CNN
 F 1 "GND" H 1400 2650 50  0000 C CNN
 F 2 "" H 1400 2800 50  0001 C CNN
@@
 	1400 2800 1400 2650
 $Comp
-L C BC?
+L C BC2
 U 1 1 59F24A6B
 P 1750 2500
-F 0 "BC?" H 1775 2600 50  0000 L CNN
+F 0 "BC2" H 1775 2600 50  0000 L CNN
 F 1 "100nF" H 1775 2400 50  0000 L CNN
 F 2 "Capacitors_SMD:C_0603" H 1788 2350 50  0001 C CNN
@@
 	1400 2650 2450 2650
 $Comp
-L C BC?
+L C BC3
 U 1 1 59F24A92
 P 2100 2500
-F 0 "BC?" H 2125 2600 50  0000 L CNN
+F 0 "BC3" H 2125 2600 50  0000 L CNN
 F 1 "100nF" H 2125 2400 50  0000 L CNN
 F 2 "Capacitors_SMD:C_0603" H 2138 2350 50  0001 C CNN
@@
 	2100 2350 2100 2200
 $Comp
-L C BC?
+L C BC4
 U 1 1 59F24B56
 P 2450 2500
-F 0 "BC?" H 2475 2600 50  0000 L CNN
+F 0 "BC4" H 2475 2600 50  0000 L CNN
 F 1 "100nF" H 2475 2400 50  0000 L CNN
 F 2 "Capacitors_SMD:C_0603" H 2488 2350 50  0001 C CNN
@@
 	1750 2350 1400 2350
 $Comp
-L +3V3 #PWR016
+L +3V3 #PWR027
 U 1 1 59F24D16
 P 1400 2200
-F 0 "#PWR016" H 1400 2050 50  0001 C CNN
+F 0 "#PWR027" H 1400 2050 50  0001 C CNN
 F 1 "+3V3" H 1400 2340 50  0000 C CNN
 F 2 "" H 1400 2200 50  0001 C CNN
@@
 $EndComp
 $Comp
-L +3V3 #PWR017
+L +3V3 #PWR028
 U 1 1 59F24D34
 P 1950 2200
-F 0 "#PWR017" H 1950 2050 50  0001 C CNN
+F 0 "#PWR028" H 1950 2050 50  0001 C CNN
 F 1 "+3V3" H 1950 2340 50  0000 C CNN
 F 2 "" H 1950 2200 50  0001 C CNN
@@
 RESET
 $Comp
-L +3V3 #PWR018
+L +3V3 #PWR029
 U 1 1 59F50B66
 P 1650 3400
-F 0 "#PWR018" H 1650 3250 50  0001 C CNN
+F 0 "#PWR029" H 1650 3250 50  0001 C CNN
 F 1 "+3V3" H 1650 3540 50  0000 C CNN
 F 2 "" H 1650 3400 50  0001 C CNN
@@
 $EndComp
 $Comp
-L D D?
+L D D1
 U 1 1 59F50B83
 P 1500 3550
-F 0 "D?" H 1500 3650 50  0000 C CNN
+F 0 "D1" H 1500 3650 50  0000 C CNN
 F 1 "CD1206-S01575" H 1500 3450 50  0000 C CNN
 F 2 "Capacitors_SMD:C_0402" H 1500 3550 50  0001 C CNN
@@
 	1500 3400 1800 3400
 $Comp
-L R R?
+L R R5
 U 1 1 59F50E25
 P 1800 3550
-F 0 "R?" V 1880 3550 50  0000 C CNN
+F 0 "R5" V 1880 3550 50  0000 C CNN
 F 1 "10k" V 1800 3550 50  0000 C CNN
 F 2 "Resistors_SMD:R_0603" V 1730 3550 50  0001 C CNN

Commit message: Initial power routing to all major chips
Connections:
- net AREF is gone; now on net +3V3: BC4.1
Changed lines of the file:
@@
 	1300 3700 1800 3700
 Connection ~ 1500 3700
+$Comp
+L +3V3 #PWR?
+U 1 1 59FCA8A7
+P 2600 2350
+F 0 "#PWR?" H 2600 2200 50  0001 C CNN
+F 1 "+3V3" H 2600 2490 50  0000 C CNN
+F 2 "" H 2600 2350 50  0001 C CNN
+F 3 "" H 2600 2350 50  0001 C CNN
+	1    2600 2350
+	1    0    0    -1
+$EndComp
 $EndSCHEMATC
