File: microquad-v1/ble.sch (KiCad schematic (older format))
At the start: 7 parts, among them U5 RT9818A-18GV

Commit message: Added layout for transistor
Parts:
- D4: footprint (none) -> LEDs:LED_0805
Changed lines of the file:
@@
 	4725 4175 5275 4175
 $Comp
-L GND #PWR42
+L GND #PWR040
 U 1 1 59F5B056
 P 5950 4225
-F 0 "#PWR42" H 5950 3975 50  0001 C CNN
+F 0 "#PWR040" H 5950 3975 50  0001 C CNN
 F 1 "GND" H 5950 4075 50  0000 C CNN
 F 2 "" H 5950 4225 50  0001 C CNN
@@
 $EndComp
 $Comp
-L GND #PWR39
+L GND #PWR041
 U 1 1 59F5B05C
 P 4225 4800
-F 0 "#PWR39" H 4225 4550 50  0001 C CNN
+F 0 "#PWR041" H 4225 4550 50  0001 C CNN
 F 1 "GND" H 4225 4650 50  0000 C CNN
 F 2 "" H 4225 4800 50  0001 C CNN
@@
 $EndComp
 $Comp
-L GND #PWR40
+L GND #PWR042
 U 1 1 59F5B072
 P 4850 4600
-F 0 "#PWR40" H 4850 4350 50  0001 C CNN
+F 0 "#PWR042" H 4850 4350 50  0001 C CNN
 F 1 "GND" H 4850 4450 50  0000 C CNN
 F 2 "" H 4850 4600 50  0001 C CNN
@@
 Connection ~ 6000 2225
 $Comp
-L GND #PWR44
+L GND #PWR043
 U 1 1 59F5B0AC
 P 6200 2575
-F 0 "#PWR44" H 6200 2325 50  0001 C CNN
+F 0 "#PWR043" H 6200 2325 50  0001 C CNN
 F 1 "GND" H 6200 2425 50  0000 C CNN
 F 2 "" H 6200 2575 50  0001 C CNN
@@
 TX
 $Comp
-L +3V3 #PWR43
+L +3V3 #PWR044
 U 1 1 59F5C114
 P 6000 2100
-F 0 "#PWR43" H 6000 1950 50  0001 C CNN
+F 0 "#PWR044" H 6000 1950 50  0001 C CNN
 F 1 "+3V3" H 6000 2240 50  0000 C CNN
 F 2 "" H 6000 2100 50  0001 C CNN
@@
 	6000 2650 6000 2100
 $Comp
-L +3V3 #PWR41
+L +3V3 #PWR045
 U 1 1 59F5C188
 P 5025 3675
-F 0 "#PWR41" H 5025 3525 50  0001 C CNN
+F 0 "#PWR045" H 5025 3525 50  0001 C CNN
 F 1 "+3V3" H 5025 3815 50  0000 C CNN
 F 2 "" H 5025 3675 50  0001 C CNN
@@
 $EndComp
 $Comp
-L +3V3 #PWR38
+L +3V3 #PWR046
 U 1 1 59F5C240
 P 3575 4025
-F 0 "#PWR38" H 3575 3875 50  0001 C CNN
+F 0 "#PWR046" H 3575 3875 50  0001 C CNN
 F 1 "+3V3" H 3575 4165 50  0000 C CNN
 F 2 "" H 3575 4025 50  0001 C CNN
@@
 $EndComp
 $Comp
-L +3V3 #PWR45
+L +3V3 #PWR047
 U 1 1 59F5C2DF
 P 7150 2900
-F 0 "#PWR45" H 7150 2750 50  0001 C CNN
+F 0 "#PWR047" H 7150 2750 50  0001 C CNN
 F 1 "+3V3" H 7150 3040 50  0000 C CNN
 F 2 "" H 7150 2900 50  0001 C CNN
@@
 F 0 "D4" H 7150 3550 50  0000 C CNN
 F 1 "LED" H 7150 3350 50  0000 C CNN
-F 2 "" H 7150 3450 50  0001 C CNN
+F 2 "LEDs:LED_0805" H 7150 3450 50  0001 C CNN
 F 3 "" H 7150 3450 50  0001 C CNN
 	1    7150 3450
