File: microquad-v1/ble.sch (KiCad schematic (older format))
At the start: 7 parts, among them U5 RT9818A-18GV

Commit message: Finished in-class work 10/2
Parts:
- U5: value RT9818A-18GV -> MAX6333UR18D3
Changed lines of the file:
@@
 P 4225 4275
 F 0 "U5" H 3925 4625 60  0000 L CNN
-F 1 "RT9818A-18GV" H 3925 4525 60  0000 L CNN
+F 1 "MAX6333UR18D3" H 3925 4525 60  0000 L CNN
 F 2 "TO_SOT_Packages_SMD:SOT-23" H 4175 4275 60  0001 C CNN
 F 3 "" H 4175 4275 60  0001 C CNN
