File: microquad-v1/motor.sch (KiCad schematic (older format))
At the start: 5 parts, among them M6 Motor_DC, Q1 Q_NMOS_GSD

Commit message: Ladybug is satisfied
Changed lines of the file:
@@
 $Descr A4 11693 8268
 encoding utf-8
-Sheet 10 15
+Sheet 13 15
 Title ""
 Date ""
@@
 AR Path="/59F7FC61/59F7E92A" Ref="#PWR053"  Part="1"
 AR Path="/59F7FFA1/59F7E92A" Ref="#PWR055"  Part="1"
-F 0 "#PWR047" H 4975 3150 50  0001 C CNN
+F 0 "#PWR053" H 4975 3150 50  0001 C CNN
 F 1 "GND" H 4975 3250 50  0000 C CNN
 F 2 "" H 4975 3400 50  0001 C CNN
@@
 AR Path="/59F7FC61/59F7E931" Ref="M4"  Part="1"
 AR Path="/59F7FFA1/59F7E931" Ref="M5"  Part="1"
-F 0 "M1" H 5075 2650 50  0000 L CNN
+F 0 "M4" H 5075 2650 50  0000 L CNN
 F 1 "Motor_DC" H 5075 2350 50  0000 L TNN
 F 2 "motor:quad_motor_v1" H 4975 2460 50  0001 C CNN
@@
 AR Path="/59F7FC61/59F7E93C" Ref="D11"  Part="1"
 AR Path="/59F7FFA1/59F7E93C" Ref="D13"  Part="1"
-F 0 "D5" H 4650 2750 50  0000 C CNN
+F 0 "D11" H 4650 2750 50  0000 C CNN
 F 1 "BAS521LP-7" H 4650 2550 50  0000 C CNN
 F 2 "Diodes_SMD:D_SOD-123F" H 4650 2650 50  0001 C CNN
@@
 AR Path="/59F7FC61/59F7E943" Ref="D12"  Part="1"
 AR Path="/59F7FFA1/59F7E943" Ref="D14"  Part="1"
-F 0 "D6" H 5300 3300 50  0000 C CNN
+F 0 "D12" H 5300 3300 50  0000 C CNN
 F 1 "DNP" H 5300 3100 50  0000 C CNN
 F 2 "Diodes_SMD:D_2114" H 5300 3200 50  0001 C CNN
@@
 AR Path="/59F7FC61/59F80E77" Ref="C8"  Part="1"
 AR Path="/59F7FFA1/59F80E77" Ref="C9"  Part="1"
-F 0 "C5" H 4325 2675 50  0000 L CNN
+F 0 "C8" H 4325 2675 50  0000 L CNN
 F 1 "10uF" H 4325 2475 50  0000 L CNN
 F 2 "Capacitors_SMD:C_0805" H 4338 2425 50  0001 C CNN
@@
 AR Path="/59F7FC61/59F80F77" Ref="#PWR054"  Part="1"
 AR Path="/59F7FFA1/59F80F77" Ref="#PWR056"  Part="1"
-F 0 "#PWR048" H 4300 2475 50  0001 C CNN
+F 0 "#PWR054" H 4300 2475 50  0001 C CNN
 F 1 "GND" H 4300 2575 50  0000 C CNN
 F 2 "" H 4300 2725 50  0001 C CNN
@@
 AR Path="/59F7FFA1/59F918D5" Ref="Q5"  Part="1"
 AR Path="/59F7FFA4/59F918D5" Ref="Q6"  Part="1"
-F 0 "Q1" H 4750 3300 50  0000 L CNN
+F 0 "Q4" H 4750 3300 50  0000 L CNN
 F 1 "Q_NMOS_GSD" H 4450 3050 50  0000 L CNN
 F 2 "TO_SOT_Packages_SMD:SOT-23" H 5075 3300 50  0001 C CNN
